File: reTerminal_Back_Expander.kicad_pcb (KiCad board)
At the start: 2 copper layers, 130.1 x 88.7 mm, 6 parts

Commit message: Add FX23 footprint
Parts:
- added J1: Hirose-FX23-100-reTerminal, local:FX23-100S, B.Cu at (0.14, 5.40)
- moved REF** 8.28 mm to (61.0, 37.0)
- moved REF** 8.28 mm to (-61.0, -37.0)
- moved REF** 8.28 mm to (61.0, -37.0)
- moved REF** 8.28 mm to (-61.0, 37.0)
- moved REF** 8.28 mm to (40.9, 5.40)
- moved REF** 8.28 mm to (-40.9, 5.40)
Other:
- board text added: "reTerminal BOTTOM"
- board text added: "reTerminal LEFT"
- board text added: "reTerminal RIGHT"
- board text added: "reTerminal TOP"
